File: HW/transducer_control/kicad/kontrol_circuit.kicad_pcb (KiCad board)
At the start: 2 copper layers, 38.1 x 58.4 mm, 13 parts, among them J1 Kontrol, J2 PWR, Q1 BC517, Q2 BC516, Q3 BC517, Q4 BC516, Q5 BC517, Q6 BC517, Y1 Transducer

Commit message: Finished BAC
Parts:
- removed Y1: Transducer, Connector_Phoenix_MSTB:PhoenixContact_MSTBA_2,5_2-G-5,08_1x02_P5.08mm_Horizontal
- added J3: Conn_01x01, Connector_PinHeader_2.54mm:PinHeader_1x01_P2.54mm_Vertical, F.Cu at (190.5, 127.0)
- added J4: Conn_01x01, Connector_PinHeader_2.54mm:PinHeader_1x01_P2.54mm_Vertical, F.Cu at (190.5, 116.8)
- added R4: 1k, Resistor_THT:R_Axial_DIN0207_L6.3mm_D2.5mm_P10.16mm_Horizontal, F.Cu at (162.6, 124.5)
- added R5: 1k, Resistor_THT:R_Axial_DIN0207_L6.3mm_D2.5mm_P10.16mm_Horizontal, F.Cu at (162.6, 119.4)
- added R6: 1k, Resistor_THT:R_Axial_DIN0207_L6.3mm_D2.5mm_P10.16mm_Horizontal, F.Cu at (172.7, 109.2)
- added R7: 1k, Resistor_THT:R_Axial_DIN0207_L6.3mm_D2.5mm_P10.16mm_Horizontal, F.Cu at (172.7, 114.3)
- J1: footprint Connector_Phoenix_MSTB:PhoenixContact_MSTBA_2,5_4-G-5,08_1x04_P5.08mm_Horizontal -> Connector_PinHeader_2.54mm:PinHeader_1x05_P2.54mm_Vertical
- J2: footprint Connector_Phoenix_MSTB:PhoenixContact_MSTBA_2,5_2-G-5,08_1x02_P5.08mm_Horizontal -> Connector_PinHeader_2.54mm:PinHeader_1x02_P2.54mm_Vertical
- R1, R3: value 3.9k -> 270k; footprint Resistor_THT:R_Axial_DIN0207_L6.3mm_D2.5mm_P10.16mm_Horizontal -> Resistor_THT:R_Axial_DIN0204_L3.6mm_D1.6mm_P2.54mm_Vertical
- moved J1 46.0 mm to (157.5, 124.5)
- moved Q5 37.8 mm to (175.3, 111.8), turned to 180 degrees
- moved Q3 36.1 mm to (175.3, 121.9), turned to 180 degrees
- moved Q4 34.2 mm to (177.8, 111.8), turned to 0 degrees
- moved R3 34.2 mm to (180.3, 116.8)
- moved Q2 32.3 mm to (177.8, 121.9), turned to 0 degrees
- moved Q6 31.8 mm to (175.3, 116.8), turned to 180 degrees
- moved R1 30.6 mm to (177.8, 127.0), turned to 0 degrees
- moved Q1 29.6 mm to (175.3, 127.0), turned to 180 degrees
- moved R2 27.4 mm to (180.3, 106.7)
- moved J2 23.4 mm to (165.1, 127.0)
- moved C1 19.4 mm to (188.0, 109.2), turned to 90 degrees
Connections:
- net Net-(C1-Pad1) renamed T2
- net Net-(Q2-Pad1) renamed T1
- J1 pad 1: V11 -> Earth
- J1 pad 2: V12 -> V11
- J1 pad 4: V22 -> V12
- Q1 pad 2: V11 -> Net-(Q1-Pad2)
- Q1 pad 3: Net-(Q1-Pad3) -> Earth
- Q2 pad 2: Net-(Q1-Pad1) -> Net-(Q2-Pad2)
- Q3 pad 2: V21 -> Net-(Q3-Pad2)
- Q5 pad 2: V22 -> Net-(Q5-Pad2)
- Q6 pad 1: Net-(Q4-Pad2) -> Net-(Q6-Pad1)
- Q6 pad 2: V12 -> Net-(Q6-Pad2)
- Q6 pad 3: Net-(Q6-Pad3) -> Earth
- R1 pad 1: Net-(Q1-Pad3) -> Net-(Q1-Pad1)
- R1 pad 2: Earth -> Net-(Q2-Pad2)
- R3 pad 1: Net-(Q6-Pad3) -> Net-(Q4-Pad2)
- R3 pad 2: Earth -> Net-(Q6-Pad1)
Routing:
- net V11: track 33.0 -> 7.62 mm, vias 2 -> 0
- net V21: track 27.9 -> 5.08 mm, vias 1 -> 0
- net T2: track 38.1 -> 25.4 mm
- net V12: track 20.3 -> 7.62 mm, vias 2 -> 0
- net Net-(C1-Pad2): track 17.8 -> 7.62 mm
- net Earth: track 27.9 -> 35.6 mm
- net +10V: track 27.9 -> 35.6 mm, vias 2 -> 0
- net Net-(Q6-Pad3): track 5.08 -> 0.00 mm
- net Net-(Q1-Pad3): track 5.08 -> 0.00 mm
- net Net-(Q2-Pad2): track 0.00 -> 5.08 mm
- net V22: track 15.2 -> 10.2 mm
- net Net-(Q6-Pad1): track 0.00 -> 2.54 mm
- net Net-(Q6-Pad2): track 0.00 -> 2.54 mm
- net Net-(Q5-Pad2): track 0.00 -> 2.54 mm
- net Net-(Q3-Pad2): track 0.00 -> 2.54 mm
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Other:
- board outline removed
