File: HW/transducer_control/kicad/kontrol_circuit.kicad_sch (KiCad schematic)
At the start: 13 parts, among them Q1 BC517, Q2 BC516, Q3 BC517, Q4 BC516, Q5 BC517

Commit message: Finished BAC
Parts:
- removed J1: (no value), symbol Connector_Generic:Conn_01x04
- removed Y1: (no value), symbol Device:Crystal
- added J1: Kontrol, Connector_PinHeader_2.54mm:PinHeader_1x05_P2.54mm_Vertical, symbol Connector_Generic:Conn_01x05
- added J3, J4: Conn_01x01, Connector_PinHeader_2.54mm:PinHeader_1x01_P2.54mm_Vertical, symbol Connector_Generic:Conn_01x01
- added R4, R5, R6, R7: 1k, Resistor_THT:R_Axial_DIN0207_L6.3mm_D2.5mm_P10.16mm_Horizontal, symbol Device:R
- C1: value (none) -> 10μ; footprint (none) -> Capacitor_THT:CP_Radial_D5.0mm_P2.50mm
- J2: value (none) -> PWR; footprint (none) -> Connector_PinHeader_2.54mm:PinHeader_1x02_P2.54mm_Vertical
- Q1, Q2, Q3, Q4, Q5: footprint (none) -> Package_TO_SOT_THT:TO-92_Inline_Wide
- Q6: value (none) -> BC517; footprint (none) -> Package_TO_SOT_THT:TO-92_Inline_Wide
- R1, R3: value (none) -> 270k; footprint (none) -> Resistor_THT:R_Axial_DIN0204_L3.6mm_D1.6mm_P2.54mm_Vertical
- R2: value (none) -> 1k; footprint (none) -> Resistor_THT:R_Axial_DIN0207_L6.3mm_D2.5mm_P10.16mm_Horizontal
Connections:
- net Earth: now also Q1.3 (E), Q6.3 (E), J1.1 (Pin_1); no longer R1.2, R3.2
- net V11: now also J1.2 (Pin_2), R4.1; no longer Q1.2 (B)
- net V12: now also J1.4 (Pin_4), R7.2; no longer Q6.2 (B)
- net V21: now also J1.3 (Pin_3), R5.1; no longer Q3.2 (B)
- net V22: now also J1.5 (Pin_5), R6.2; no longer Q5.2 (B)
- net T1: now reaches Q2.1 (C), Q3.1 (C)
- net T1: now also J3.1 (Pin_1)
- net T2: now reaches C1.1, Q4.1 (C), Q5.1 (C)
- net T2: now also J4.1 (Pin_1)
- net at R1.1: now also Q1.1 (C); no longer Q1.3 (E)
- net at Q6.1 (C): now also R3.2; no longer Q4.2 (B)
- net at R3.1: now also Q4.2 (B); no longer Q6.3 (E)
- net at Q2.2 (B): now also R1.2; no longer Q1.1 (C)
- new net: Q3.2 (B), R5.2
- new net: Q5.2 (B), R6.1
- new net: Q6.2 (B), R7.1
- new net: Q1.2 (B), R4.2
